File: Rev. 0/Eagle/C64_KernalSw_8k.brd (EAGLE design)
At the start: 22 x 45 mm, 11 parts, among them IC1 M27C512-DIP28, IC2 2364

Commit message: Silk Screen Update
Parts:
- added U$11: OPEN_SOURCE_HW, Logo:OPENHW
- added U$6: (no value), Logo:SVEN_TAG
Other:
- board text added: "3x10k"
- board text added: "http://github.com/ svenpetersen1965"
Changed lines of the file:
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@@
 <?xml version="1.0" encoding="utf-8"?>
 <!DOCTYPE eagle SYSTEM "eagle.dtd">
-<eagle version="9.2.2">
+<eagle version="9.5.2">
 <drawing>
 <settings>
@@
 <layer number="20" name="Dimension" color="24" fill="1" visible="yes" active="yes"/>
 <layer number="21" name="tPlace" color="7" fill="1" visible="yes" active="yes"/>
-<layer number="22" name="bPlace" color="7" fill="1" visible="yes" active="yes"/>
+<layer number="22" name="bPlace" color="7" fill="1" visible="no" active="yes"/>
 <layer number="23" name="tOrigins" color="15" fill="1" visible="yes" active="yes"/>
 <layer number="24" name="bOrigins" color="15" fill="1" visible="no" active="yes"/>
-<layer number="25" name="tNames" color="7" fill="1" visible="no" active="yes"/>
+<layer number="25" name="tNames" color="7" fill="1" visible="yes" active="yes"/>
 <layer number="26" name="bNames" color="7" fill="1" visible="no" active="yes"/>
-<layer number="27" name="tValues" color="7" fill="1" visible="yes" active="yes"/>
+<layer number="27" name="tValues" color="7" fill="1" visible="no" active="yes"/>
 <layer number="28" name="bValues" color="7" fill="1" visible="no" active="yes"/>
 <layer number="29" name="tStop" color="7" fill="3" visible="no" active="yes"/>
@@
 <layer number="250" name="Descript" color="7" fill="1" visible="no" active="no"/>
 <layer number="251" name="SMDround" color="7" fill="1" visible="no" active="no"/>
+<layer number="252" name="BR-BS" color="7" fill="1" visible="no" active="yes"/>
+<layer number="253" name="BR-LS" color="7" fill="1" visible="no" active="yes"/>
 <layer number="254" name="OrgLBR" color="7" fill="1" visible="no" active="no"/>
 <layer number="255" name="Accent" color="7" fill="1" visible="yes" active="yes"/>
@@
 C64 short board</text>
 <text x="11.27125" y="3.81" size="1.1684" layer="47" ratio="12" rot="R90">Rev. 0</text>
-<text x="11.90625" y="3.81" size="1.1684" layer="21" ratio="12" rot="R90">Kernal Adapt/Sw
+<text x="9.68375" y="3.81" size="1.1684" layer="21" ratio="12" rot="R90">Kernal Adapt/Sw
 C64 long board</text>
-<text x="13.97" y="3.81" size="1.1684" layer="21" ratio="12" rot="R90">Rev. 0</text>
+<text x="11.58875" y="3.81" size="1.1684" layer="21" ratio="12" rot="R90">Rev. 0</text>
 <text x="9.8425" y="4.7625" size="1.778" layer="22" ratio="12" rot="MR90">Kernal Adapt/Sw Rev. 0
 C64 long board</text>
+<text x="6.985" y="28.2575" size="1.016" layer="25">3x10k</text>
+<text x="14.9225" y="3.81" size="1.016" layer="25" rot="R90">http://github.com/
+svenpetersen1965</text>
 </plain>
 <attributes>
@@
 </element>
 <element name="R1" library="SMD" package="0805" value="10k" x="13.6525" y="29.845" smashed="yes" rot="R180">
-<attribute name="NAME" x="13.58775" y="27.6185" size="1.016" layer="25" ratio="10"/>
+<attribute name="NAME" x="14.064" y="27.6185" size="1.016" layer="25" ratio="10"/>
 <attribute name="VALUE" x="15.24" y="30.2895" size="1.016" layer="27" ratio="10" rot="R180"/>
 </element>
@@
 <attribute name="VALUE" x="0.56125" y="36.42025" size="1.27" layer="28"/>
 </element>
+<element name="U$6" library="Logo" package="SVEN_TAG" value="" x="7.46125" y="14.76375" smashed="yes" rot="MR0"/>
+<element name="U$11" library="Logo" package="OPENHW" value="OPEN_SOURCE_HW" x="14.76375" y="20.16125" smashed="yes" rot="R90"/>
 </elements>
 <signals>
