File: Rev. 0/Eagle/C64_KernalSw_8k.sch (EAGLE design)
At the start: 6 parts, among them IC1 M27C512-DIP28, IC2 2364

Commit message: Silk Screen Update
Parts:
- added U$11: OPEN_SOURCE_HW, Logo:OPEN_SOURCE_HW
Other:
- note added: "http://github.com/svenpetersen1965"
Changed lines of the file:
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@@
 <?xml version="1.0" encoding="utf-8"?>
 <!DOCTYPE eagle SYSTEM "eagle.dtd">
-<eagle version="9.2.2">
+<eagle version="9.5.2">
 <drawing>
 <settings>
@@
 <layer number="250" name="Descript" color="7" fill="1" visible="no" active="no"/>
 <layer number="251" name="SMDround" color="7" fill="1" visible="no" active="no"/>
+<layer number="252" name="BR-BS" color="7" fill="1" visible="no" active="yes"/>
+<layer number="253" name="BR-LS" color="7" fill="1" visible="no" active="yes"/>
 <layer number="254" name="OrgLBR" color="7" fill="1" visible="no" active="no"/>
 <layer number="255" name="Accent" color="7" fill="1" visible="yes" active="yes"/>
@@
 <part name="U$15" library="!GRAFIK" deviceset="IN" device=""/>
 <part name="IC2" library="MOS" deviceset="2364" device=""/>
+<part name="U$11" library="Logo" deviceset="OPEN_SOURCE_HW" device=""/>
 </parts>
 <sheets>
@@
 <text x="276.86" y="27.94" size="2.54" layer="95">C64 Kernal Adaptor/Switch</text>
 <text x="276.86" y="22.86" size="2.54" layer="95">for long boards</text>
+<text x="279.4" y="7.62" size="2.54" layer="95">http://github.com/svenpetersen1965</text>
 </plain>
 <instances>
@@
 <attribute name="VALUE" x="193.04" y="119.38" size="1.27" layer="96"/>
 </instance>
+<instance part="U$11" gate="G$1" x="233.68" y="10.16" smashed="yes"/>
 </instances>
 <busses>
